Commit message: more realistic bot

File: src/mybot_description/urdf/mybot.xacro (robot description, xacro)
@@ -1,23 +1,20 @@
 <?xml version='1.0'?>
-<robot name="myrobot" xmlns:xacro="http://www.ros.org/wiki/xacro">
+<robot name="myrobot"
+  xmlns:xacro="http://www.ros.org/wiki/xacro">
   <xacro:property name="cameraSize" value="0.05"/>
   <xacro:property name="cameraMass" value="0.1"/>
-  <xacro:include filename="$(find mybot_description)/urdf/mybot.gazebo" />
-  <xacro:include filename="$(find mybot_description)/urdf/materials.xacro" />
-  <xacro:include filename="$(find mybot_description)/urdf/macros.xacro" />
+  <xacro:include filename="$(find ugv_description)/urdf/mybot.gazebo" />
+  <xacro:include filename="$(find ugv_description)/urdf/materials.xacro" />
+  <xacro:include filename="$(find ugv_description)/urdf/macros.xacro" />
   <link name='chassis'>
-    <pose>0 0 0.1 0 0 0</pose>
+    <pose>0 0 0.5 0 0 0</pose>
     <inertial>
       <mass value="15.0"/>
       <origin xyz="0.0 0 0.1" rpy=" 0 0 0"/>
-      <inertia
-          ixx="0.1" ixy="0" ixz="0"
-          iyy="0.1" iyz="0"
-          izz="0.1"
-      />
+      <inertia ixx="0.1" ixy="0" ixz="0" iyy="0.1" iyz="0" izz="0.1" />
     </inertial>
     <collision name='collision'>
       <geometry>
-        <box size=".4 .2 .1"/>
+        <box size=".9 .6 .4"/>
       </geometry>
     </collision>
@@ -25,11 +22,11 @@
       <origin xyz="0 0 0" rpy=" 0 0 0"/>
       <geometry>
-        <box size=".4 .2 .1"/>
+        <box size=".9 .6 .4"/>
       </geometry>
     </visual>
     <collision name='caster_collision'>
-      <origin xyz="-0.15 0 -0.05" rpy=" 0 0 0"/>
+      <origin xyz="-0.15 0 -0.18" rpy=" 0 0 0"/>
       <geometry>
-        <sphere radius="0.05"/>
+        <sphere radius="0.15"/>
       </geometry>
       <surface>
@@ -45,29 +42,7 @@
     </collision>
     <visual name='caster_visual'>
-      <origin xyz="-0.15 0 -0.05" rpy=" 0 0 0"/>
+      <origin xyz="-0.15 0 -0.18" rpy=" 0 0 0"/>
       <geometry>
-        <sphere radius="0.05"/>
-      </geometry>
-    </visual>
-    <collision name='caster_front_collision'>
-      <origin xyz="0.15 0 -0.05" rpy=" 0 0 0"/>
-      <geometry>
-        <sphere radius="0.05"/>
-      </geometry>
-      <surface>
-        <friction>
-          <ode>
-            <mu>0</mu>
-            <mu2>0</mu2>
-            <slip1>1.0</slip1>
-            <slip2>1.0</slip2>
-          </ode>
-        </friction>
-      </surface>
-    </collision>
-    <visual name='caster_front_visual'>
-      <origin xyz="0.15 0 -0.05" rpy=" 0 0 0"/>
-      <geometry>
-        <sphere radius="0.05"/>
+        <sphere radius="0.15"/>
       </geometry>
     </visual>
@@ -78,5 +53,5 @@
       <origin xyz="0 0 0" rpy="0 1.5707 1.5707"/>
       <geometry>
-        <cylinder radius="0.1" length="0.05"/>
+        <cylinder radius="0.15" length="0.08"/>
       </geometry>
     </collision>
@@ -84,5 +59,5 @@
       <origin xyz="0 0 0" rpy="0 1.5707 1.5707"/>
       <geometry>
-        <cylinder radius="0.1" length="0.05"/>
+        <cylinder radius="0.15" length="0.08"/>
       </geometry>
     </visual>
@@ -90,8 +65,5 @@
       <origin xyz="0 0 0" rpy="0 1.5707 1.5707"/>
       <mass value="5"/>
-      <inertia
-        ixx=".1" ixy="0.0" ixz="0.0"
-        iyy=".1" iyz="0.0"
-        izz=".1"/>
+      <inertia ixx=".1" ixy="0.0" ixz="0.0" iyy=".1" iyz="0.0" izz=".1"/>
     </inertial>
   </link>
@@ -101,5 +73,5 @@
       <origin xyz="0 0 0" rpy="0 1.5707 1.5707"/>
       <geometry>
-        <cylinder radius="0.1" length="0.05"/>
+        <cylinder radius="0.15" length="0.08"/>
       </geometry>
     </collision>
@@ -107,5 +79,5 @@
       <origin xyz="0 0 0" rpy="0 1.5707 1.5707"/>
       <geometry>
-        <cylinder radius="0.1" length="0.05"/>
+        <cylinder radius="0.15" length="0.08"/>
       </geometry>
     </visual>
@@ -113,12 +85,9 @@
       <origin xyz="0 0 0" rpy="0 1.5707 1.5707"/>
       <mass value="5"/>
-      <inertia
-        ixx=".1" ixy="0.0" ixz="0.0"
-        iyy=".1" iyz="0.0"
-        izz=".1"/>
+      <inertia ixx=".1" ixy="0.0" ixz="0.0" iyy=".1" iyz="0.0" izz=".1"/>
     </inertial>
   </link>
   <joint type="continuous" name="left_wheel_hinge">
-    <origin xyz="0 0.15 0" rpy="0 0 0"/>
+    <origin xyz="0.3 0.35 -0.15" rpy="0 0 0"/>
     <!--origin xyz="0.1 0.13 0" rpy="0 1.5707 1.5707"/-->
     <child link="left_wheel"/>
@@ -129,5 +98,5 @@
   </joint>
   <joint type="continuous" name="right_wheel_hinge">
-    <origin xyz="0 -0.15 0" rpy="0 0 0"/>
+    <origin xyz="0.3 -0.35 -0.15" rpy="0 0 0"/>
     <!--origin xyz="0.1 -0.13 0" rpy="0 1.5707 1.5707"/-->
     <child link="right_wheel"/>
@@ -139,5 +108,5 @@
   <link name="camera">
     <collision>
-      <origin xyz="0 0 0" rpy="0 0 0"/>
+      <origin xyz="0 0 0.5" rpy="0 0 0"/>
       <geometry>
         <box size="${cameraSize} ${cameraSize} ${cameraSize}"/>
@@ -145,5 +114,5 @@
     </collision>
     <visual>
-      <origin xyz="0 0 0" rpy="0 0 0"/>
+      <origin xyz="0 0 0.5" rpy="0 0 0"/>
       <geometry>
         <box size="${cameraSize} ${cameraSize} ${cameraSize}"/>
@@ -153,5 +122,5 @@
     <inertial>
       <mass value="${cameraMass}" />
-      <origin xyz="0 0 0" rpy="0 0 0"/>
+      <origin xyz="0 0 0.5" rpy="0 0 0"/>
       <box_inertia m="${cameraMass}" x="${cameraSize}" y="${cameraSize}" z="${cameraSize}" />
       <inertia ixx="1e-6" ixy="0" ixz="0" iyy="1e-6" iyz="0" izz="1e-6" />
@@ -159,12 +128,39 @@
   </link>
   <joint name="camera_joint" type="fixed">
-    <axis xyz="0 1 0" />
-    <origin xyz=".2 0 0" rpy="0 0 0"/>
-    <parent link="chassis"/>
+    <axis xyz="0 0 0" />
+    <origin xyz="0 0 0.3" rpy="0 0 0"/>
+    <parent link="camera_stick"/>
     <child link="camera"/>
   </joint>
+  <link name="camera_stick">
+    <collision>
+      <origin xyz="0 0 0" rpy="0 0 0"/>
+      <geometry>
+        <box size="${cameraSize/2} ${cameraSize/2} 1.37"/>
+      </geometry>
+    </collision>
+    <visual>
+      <origin xyz="0 0 0.1" rpy="0 0 0"/>
+      <geometry>
+        <box size="${cameraSize/2} ${cameraSize/2} 1.37"/>
+      </geometry>
+      <material name="black"/>
+    </visual>
+    <inertial>
+      <mass value="${cameraMass}" />
+      <origin xyz="0 0 0.1" rpy="0 0 0"/>
+      <box_inertia m="${cameraMass}" x="${cameraSize}" y="${cameraSize}" z="${cameraSize}" />
+      <inertia ixx="1e-6" ixy="0" ixz="0" iyy="1e-6" iyz="0" izz="1e-6" />
+    </inertial>
+  </link>
+  <joint name="camera_stick_joint" type="fixed">
+    <axis xyz="0 0 0" />
+    <origin xyz="0.2 0 0.786" rpy="0 0 0"/>
+    <parent link="chassis"/>
+    <child link="camera_stick"/>
+  </joint>
   <joint name="hokuyo_joint" type="fixed">
-    <axis xyz="0 1 0" />
-    <origin xyz=".15 0 .1" rpy="0 0 0"/>
+    <axis xyz="0 0 0" />
+    <origin xyz=".45 0 .2" rpy="0 0 0"/>
     <parent link="chassis"/>
     <child link="hokuyo"/>
@@ -175,5 +171,5 @@
       <origin xyz="0 0 0" rpy="0 0 0"/>
       <geometry>
-    <box size="0.1 0.1 0.1"/>
+        <box size="0.1 0.1 0.1"/>
       </geometry>
     </collision>
@@ -181,5 +177,5 @@
       <origin xyz="0 0 0" rpy="0 0 0"/>
       <geometry>
-        <mesh filename="package://mybot_description/meshes/hokuyo.dae"/>
+        <mesh filename="package://ugv_description/meshes/hokuyo.dae"/>
       </geometry>
     </visual>

Commit message: Remove GPU lasers & use laser_plugin

File: src/mybot_description/urdf/mybot.xacro (robot description, xacro)
@@ -4,7 +4,7 @@
   <xacro:property name="cameraSize" value="0.05"/>
   <xacro:property name="cameraMass" value="0.1"/>
-  <xacro:include filename="$(find ugv_description)/urdf/mybot.gazebo" />
-  <xacro:include filename="$(find ugv_description)/urdf/materials.xacro" />
-  <xacro:include filename="$(find ugv_description)/urdf/macros.xacro" />
+  <xacro:include filename="$(find mybot_description)/urdf/mybot.gazebo" />
+  <xacro:include filename="$(find mybot_description)/urdf/materials.xacro" />
+  <xacro:include filename="$(find mybot_description)/urdf/macros.xacro" />
   <link name='chassis'>
     <pose>0 0 0.5 0 0 0</pose>
@@ -160,12 +160,12 @@
     <child link="camera_stick"/>
   </joint>
-  <joint name="hokuyo_joint" type="fixed">
+  <joint name="laser_joint" type="fixed">
     <axis xyz="0 0 0" />
     <origin xyz=".45 0 .2" rpy="0 0 0"/>
     <parent link="chassis"/>
-    <child link="hokuyo"/>
+    <child link="laser"/>
   </joint>
   <!-- Hokuyo Laser -->
-  <link name="hokuyo">
+  <link name="laser">
     <collision>
       <origin xyz="0 0 0" rpy="0 0 0"/>
@@ -177,5 +177,5 @@
       <origin xyz="0 0 0" rpy="0 0 0"/>
       <geometry>
-        <mesh filename="package://ugv_description/meshes/hokuyo.dae"/>
+        <mesh filename="package://mybot_description/meshes/hokuyo.dae"/>
       </geometry>
     </visual>
