Commit message: create dummy frame for ROS URDF

File: src/mybot_description/urdf/mybot.urdf.xacro (robot description, xacro)
@@ -9,4 +9,6 @@
   <xacro:include filename="$(find mybot_description)/urdf/gps.urdf.xacro" />
   <xacro:gps parent="chassis"></xacro:gps>
+  <link name="dummy">
+  </link>
   <link name='chassis'>
     <pose>0 0 0.5 0 0 0</pose>
@@ -72,4 +74,8 @@
     </visual-->
   </link>
+  <joint name="dummy_joint" type="fixed">
+  	<parent link="dummy"/>
+  	<child link="chassis"/>
+  </joint>
   <link name="left_wheel">
     <!--origin xyz="0.1 0.13 0.1" rpy="0 1.5707 1.5707"/-->

Commit message: Change base frame id to base_link

File: src/mybot_description/urdf/mybot.urdf.xacro (robot description, xacro)
@@ -8,8 +8,8 @@
   <xacro:include filename="$(find mybot_description)/urdf/macros.xacro" />
   <xacro:include filename="$(find mybot_description)/urdf/gps.urdf.xacro" />
-  <xacro:gps parent="chassis"></xacro:gps>
+  <xacro:gps parent="base_link"></xacro:gps>
   <link name="dummy">
   </link>
-  <link name='chassis'>
+  <link name='base_link'>
     <pose>0 0 0.5 0 0 0</pose>
     <inertial>
@@ -23,5 +23,5 @@
       </geometry>
     </collision>
-    <visual name='chassis_visual'>
+    <visual name='base_link_visual'>
       <origin xyz="0 0 0" rpy=" 0 0 0"/>
       <geometry>
@@ -76,5 +76,5 @@
   <joint name="dummy_joint" type="fixed">
   	<parent link="dummy"/>
-  	<child link="chassis"/>
+  	<child link="base_link"/>
   </joint>
   <link name="left_wheel">
@@ -138,5 +138,5 @@
     <!--origin xyz="0.1 0.13 0" rpy="0 1.5707 1.5707"/-->
     <child link="left_wheel"/>
-    <parent link="chassis"/>
+    <parent link="base_link"/>
     <axis xyz="0 1 0" rpy="0 0 0"/>
     <limit effort="10000" velocity="1000"/>
@@ -147,5 +147,5 @@
     <!--origin xyz="0.1 -0.13 0" rpy="0 1.5707 1.5707"/-->
     <child link="right_wheel"/>
-    <parent link="chassis"/>
+    <parent link="base_link"/>
     <axis xyz="0 1 0" rpy="0 0 0"/>
     <limit effort="10000" velocity="1000"/>
@@ -203,5 +203,5 @@
     <axis xyz="0 0 0" />
     <origin xyz="0.2 0 0.786" rpy="0 0 0"/>
-    <parent link="chassis"/>
+    <parent link="base_link"/>
     <child link="camera_stick"/>
   </joint>
@@ -209,5 +209,5 @@
     <axis xyz="0 0 0" />
     <origin xyz=".45 0 .25" rpy="0 0 0"/>
-    <parent link="chassis"/>
+    <parent link="base_link"/>
     <child link="laser"/>
   </joint>
